File: RPI-Lora-Gateway-Shield.sch (EAGLE design)
At the start: 58 parts, among them J1 GROVE, J10 CON_TERMINAL_BLOCK_02-5MM, J11 JUMPER_1X30805, J12 JUMPER_1X30805, J13 GROVE I2C, J14 2.54_I2C, J15 POWER_JACKPTH, J4 RASPBERRYPI-40-PIN-GPIO, J5 DHTxx, J6 2.54_I2C, J7 2.54_I2C, J8 CON_TERMINAL_BLOCK_02-5MM, J9 CON_TERMINAL_BLOCK_02-5MM

Commit message: Bump to Version 1.1
Parts:
- removed GROVE: GROVE I2C, Connector -2016:GROVE-CONNECTOR-DIP(4P-2.0)
- removed H1, H2, H3, H4, H5, H6: STAND-OFF, SparkFun-Electromechanical:STAND-OFF
- removed J$1: ANTENNATINY, _c2h:ANTENNATINY
- added J16: 2.54_PWR, _c2h:CON_HEADER_1X04'NO_LOCK'
- added U$3: ANTENNA-UFL, _c2h:ANTENNA-UFL
- added U$8: DC-BREAKOUTFIXED, _c2h:DC-BREAKOUTFIXED
- JP1, JP2: device microbuilder:JUMPER3 -> microbuilder:JUMPER2
Connections:
- removed net N$14: D3.A, D4.A, J15.PWR, J8.1
- new net 5V-PI: J4.5V@2, J4.5V@4, JP1.2
- new net SPI_SEL: J12.2, U$2.SEL
- new net VIN: D3.A, D4.A, J15.PWR, J16.2, J16.3, J8.1, JP2.1
- net +5V: now also J16.4, JP1.1, JP2.2, U$8.VOUT; no longer J4.5V@2, J4.5V@4
- net 3V3: no longer GROVE.3, R11.1, R12.1
- net GND: now also J16.1, R11.1, R12.1, U$3.GND@0, U$3.GND@1, U$8.GND; no longer GROVE.4, J$1.GND@0, J$1.GND@1, J$1.GND@2, J$1.GND@3
- net N$28: now also U$8.VIN
- net N$29: now also U$3.SIGNAL; no longer J$1.SIGNAL
- net SCL: no longer GROVE.1
- net SDA: no longer GROVE.2
- net SPI_CE0: no longer JP1.1, JP2.1
- net SPI_CE1: no longer JP1.3, JP2.3
- net SPI_SS: no longer J12.2, JP1.2, JP2.2, U$2.SEL
Other:
- note added: "Close JP1 to: - power ic880a from RPI Power (USB Connector) - or power PI from ic880a power"
- note added: "Close JP2 if Power Supply is already 5V and no using the DC/DC step down"
- moved on the sheet: D3, DC/DC, J15, J8, R11

Commit message: Bump to V1.2
Parts:
- added FTDI: CON_HEADER_1X06-PTH, _c2h:CON_HEADER_1X06-PTH
- added SW1: (no value), adafruit:SWITCH_PUSHBUTTONEVQ-PE
- added U$11: OKI-78SR, _c2h:DCDC_OKI-78SRHORZ
Connections:
- net GPIO35 renamed GPIO26
- removed net N$28: D3.C, D4.C, DC/DC.VIN, U$8.VIN
- new net N$14: D3.C, D4.C, DC/DC.VIN, U$11.VI, U$8.VIN
- new net RXI: FTDI.4, J4.RXI
- new net TXO: FTDI.5, J4.TXO
- net +5V: now also U$11.VO
- net 3V3: now also SW1.P$2
- net GND: now also FTDI.1, U$11.GND
- net GPIO19: now also SW1.P$1
Other:
- note added: "FTDI_GND"
- note added: "FTDI_RXD"
- note added: "FTDI_TXD"
- note added: "push SW1 to shutdown GW"
- moved on the sheet: J10, J9, JP2
